File: KiCAD/SawVCO/SawVCO.sch (KiCad schematic (older format))
At the start: 42 parts, among them J1 PWR_IN, J10 Saw_Out, J2 Liner_FM, J3 PWR_OUT, J4 I_Ref, J5 I_Sink, J6 TP_GND, J7 Sync_In, J8 Saw_Out, J9 Saw_Out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

Commit message: Update
Parts:
- C11: footprint Capacitor_THT:C_Disc_D3.0mm_W1.6mm_P2.50mm -> Capacitor_THT:C_Disc_D4.3mm_W1.9mm_P5.00mm
- RV1: value 5k -> 10k; footprint myfootprint:Potentiometer_Bourns_3362P_Vertical -> Potentiometer_THT:Potentiometer_Bourns_3296W_Vertical
Changed lines of the file:
@@
 F 0 "C11" V 6798 1950 50  0000 C CNN
 F 1 "100p" V 6889 1950 50  0000 C CNN
-F 2 "Capacitor_THT:C_Disc_D3.0mm_W1.6mm_P2.50mm" H 7088 1800 50  0001 C CNN
+F 2 "Capacitor_THT:C_Disc_D4.3mm_W1.9mm_P5.00mm" H 7088 1800 50  0001 C CNN
 F 3 "~" H 7050 1950 50  0001 C CNN
 	1    7050 1950
@@
 P 5000 2900
 F 0 "RV1" H 4930 2946 50  0000 R CNN
-F 1 "5k" H 4930 2855 50  0000 R CNN
-F 2 "myfootprint:Potentiometer_Bourns_3362P_Vertical" H 5000 2900 50  0001 C CNN
+F 1 "10k" H 4930 2855 50  0000 R CNN
+F 2 "Potentiometer_THT:Potentiometer_Bourns_3296W_Vertical" H 5000 2900 50  0001 C CNN
 F 3 "~" H 5000 2900 50  0001 C CNN
 	1    5000 2900
